File: Hardware/edafru_v1alpha/mcu.kicad_sch (KiCad schematic)
At the start: 34 parts, among them J2 ICSP, U5 PIC18F25K80_ISS, U7 AT24CS02-SSHM, Y1 8.000 MHz

Commit message: the hardware is developing..
Connections:
- net I2C_SCL: no longer R56.1
- net I2C_SDA: no longer R57.1
- net MEM_WP: no longer R58.1
- new net SPI_SCK: R56.1
- new net SPI_SDI: R57.1
- new net SPI_SDO: R58.1
Changed lines of the file:
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@@
+	(wire
+		(pts
+			(xy 177.8 130.81) (xy 193.04 130.81)
+		)
+		(stroke
+			(width 0)
+			(type default)
+		)
+	)
 	(wire
 		(pts
@@
 	(wire
 		(pts
+			(xy 177.8 135.89) (xy 193.04 135.89)
+		)
+		(stroke
+			(width 0)
+			(type default)
+		)
+	)
+	(wire
+		(pts
 			(xy 170.18 100.33) (xy 161.29 100.33)
 		)
@@
 	(wire
 		(pts
+			(xy 177.8 133.35) (xy 193.04 133.35)
+		)
+		(stroke
+			(width 0)
+			(type default)
+		)
+	)
+	(wire
+		(pts
 			(xy 193.04 100.33) (xy 177.8 100.33)
 		)
@@
 	(wire
 		(pts
-			(xy 193.04 128.27) (xy 177.8 128.27)
-		)
-		(stroke
-			(width 0)
-			(type default)
-		)
-	)
-	(wire
-		(pts
 			(xy 167.64 52.07) (xy 152.4 52.07)
 		)
@@
 	(wire
 		(pts
-			(xy 193.04 133.35) (xy 177.8 133.35)
-		)
-		(stroke
-			(width 0)
-			(type default)
-		)
-	)
-	(wire
-		(pts
 			(xy 102.87 134.62) (xy 102.87 128.27)
 		)
@@
 	(wire
 		(pts
-			(xy 193.04 138.43) (xy 177.8 138.43)
-		)
-		(stroke
-			(width 0)
-			(type default)
-		)
-	)
-	(wire
-		(pts
 			(xy 102.87 128.27) (xy 120.65 128.27)
 		)
@@
 	(wire
 		(pts
-			(xy 193.04 135.89) (xy 177.8 135.89)
-		)
-		(stroke
-			(width 0)
-			(type default)
-		)
-	)
-	(wire
-		(pts
 			(xy 170.18 115.57) (xy 161.29 115.57)
 		)
@@
 	(wire
 		(pts
+			(xy 177.8 138.43) (xy 193.04 138.43)
+		)
+		(stroke
+			(width 0)
+			(type default)
+		)
+	)
+	(wire
+		(pts
 			(xy 167.64 67.31) (xy 167.64 69.85)
 		)
@@
 	(wire
 		(pts
+			(xy 177.8 128.27) (xy 193.04 128.27)
+		)
+		(stroke
+			(width 0)
+			(type default)
+		)
+	)
+	(wire
+		(pts
 			(xy 109.22 133.35) (xy 109.22 146.05)
 		)
@@
 		(pts
 			(xy 170.18 107.95) (xy 161.29 107.95)
-		)
-		(stroke
-			(width 0)
-			(type default)
-		)
-	)
-	(wire
-		(pts
-			(xy 193.04 130.81) (xy 177.8 130.81)
 		)
 		(stroke
@@
 		)
 	)
-	(label "MEM_WP"
-		(at 189.23 133.35 180)
+	(label "SPI_SDO"
+		(at 193.04 133.35 180)
 		(effects
 			(font
@@
 		)
 	)
-	(label "I2C_SDA"
-		(at 189.23 130.81 180)
+	(label "SPI_SDI"
+		(at 193.04 130.81 180)
 		(effects
 			(font
@@
 	)
 	(label "LIN_RX"
-		(at 181.61 138.43 0)
-		(effects
-			(font
-				(size 1.27 1.27)
-			)
-			(justify left bottom)
+		(at 191.77 138.43 180)
+		(effects
+			(font
+				(size 1.27 1.27)
+			)
+			(justify right bottom)
 		)
 	)
@@
 		)
 	)
-	(label "I2C_SCL"
-		(at 189.23 128.27 180)
+	(label "SPI_SCK"
+		(at 193.04 128.27 180)
 		(effects
 			(font
@@
 	)
 	(label "LIN_TX"
-		(at 181.61 135.89 0)
-		(effects
-			(font
-				(size 1.27 1.27)
-			)
-			(justify left bottom)
-		)
-	)
+		(at 191.77 135.89 180)
+		(effects
+			(font
+				(size 1.27 1.27)
+			)
+			(justify right bottom)
+		)
+	)
