File: Hardware/edafru_v1alpha/wideband.kicad_sch (KiCad schematic)
At the start: 40 parts, among them Q6 MMBT2222A, U13 LM324A, U15 CJ125

Commit message: the hardware is developing..
Parts:
- added R167: 10K, Resistor_SMD:R_0603_1608Metric_Pad0.98x0.95mm_HandSolder, symbol Device:R
- added U16: CJ125, CJ125:SO24W, symbol CJ125:CJ125
Connections:
- net BUS_SP1_MISO: now also U16.14 (MISO)
- net BUS_SPI1_MOSI: now also U16.15 (MOSI)
- net BUS_SPI1_SCK: now also U16.13 (SCK)
- net GND: now also R167.1
- net WIDEBAND_UA: now also U16.21 (UA)
- net WIDEBAND_UR: now also U16.12 (UR)
- new net: R167.2, U16.5 (OSZ)
- new net BUS_SPI1_NSS: U16.16 (~{SS})
- new net CJ125_DIAHD: U16.7 (DIAHD)
- new net CJ125_DIAHG: U16.6 (DIAHG)
Other:
- moved on the sheet: C71, C72, C73, C74, C75, C76, C77, C78, C79, Q6, R154, R155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
